Commit message: edit description of robot :> wheel size, chasis size, and caster size , and all of positions 3 items mentioned before

File: description/robot_core.xacro (robot description, xacro)
@@ -2,20 +2,27 @@
 <robot xmlns:xacro="http://www.ros.org/wiki/xacro" >
     <xacro:include filename="inertial_macros.xacro"/>
-    <xacro:property name="chassis_length" value="0.335"/>
-    <xacro:property name="chassis_width" value="0.265"/>
-    <xacro:property name="chassis_height" value="0.138"/>
+    <xacro:property name="chassis_length" value="0.1688"/>
+    <xacro:property name="chassis_width" value="0.112"/>
+    <xacro:property name="chassis_height" value="0.05"/>
     <xacro:property name="chassis_mass" value="1.0"/>
     <xacro:property name="wheel_radius" value="0.033"/>
-    <xacro:property name="wheel_thickness" value="0.026"/>
+    <xacro:property name="wheel_thickness" value="0.028"/>
     <xacro:property name="wheel_mass" value="0.05"/>
-    <xacro:property name="wheel_offset_x" value="0.226"/>
-    <xacro:property name="wheel_offset_y" value="0.1485"/>
-    <xacro:property name="wheel_offset_z" value="0.01"/>
-    <xacro:property name="caster_wheel_radius" value="0.01"/>
+    <xacro:property name="wheel_offset_x" value="0.145"/>
+    <xacro:property name="wheel_offset_y" value="0.0675"/>
+    <xacro:property name="wheel_offset_z" value="0.035"/>
+    <xacro:property name="caster_wheel_radius" value="0.033"/>
     <xacro:property name="caster_wheel_mass" value="0.01"/>
-    <xacro:property name="caster_wheel_offset_x" value="0.075"/>
-    <xacro:property name="caster_wheel_offset_z" value="${wheel_offset_z - wheel_radius + caster_wheel_radius}"/>
+    <xacro:property name="caster_wheel_offset_x" value="0.025"/>
+    <!-- <xacro:property name="caster_wheel_offset_z" value="${wheel_offset_z - wheel_radius + caster_wheel_radius}"/> -->
+    <xacro:property name="caster_wheel_offset_z" value="${-caster_wheel_radius}"/>
     <material name="white">
         <color rgba="1 1 1 1"/>
+    </material>
+    <material name="yellow">
+        <color rgba="0.96 0.89 0.15 1"/>
+    </material>
+    <material name="green">
+        <color rgba="0.1 0.7 0.5 1"/>
     </material>
     <material name="orange">
@@ -46,5 +53,5 @@
         <parent link="base_link"/>
         <child link="chassis"/>
-        <origin xyz="${-wheel_offset_x} 0 ${-wheel_offset_z}"/>
+        <origin xyz="${-wheel_offset_x} 0 ${wheel_offset_z}"/>
     </joint>
     <link name="chassis">
@@ -54,5 +61,5 @@
                 <box size="${chassis_length} ${chassis_width} ${chassis_height}"/>
             </geometry>
-            <material name="orange"/>
+            <material name="green"/>
         </visual>
         <collision>
@@ -81,5 +88,5 @@
                 <cylinder radius="${wheel_radius}" length="${wheel_thickness}"/>
             </geometry>
-            <material name="blue"/>
+            <material name="yellow"/>
         </visual>
         <collision>
@@ -107,5 +114,5 @@
                 <cylinder radius="${wheel_radius}" length="${wheel_thickness}"/>
             </geometry>
-            <material name="blue"/>
+            <material name="yellow"/>
         </visual>
         <collision>

Commit message: change some robot description move both drive and caster wheel to the correct position

File: description/robot_core.xacro (robot description, xacro)
@@ -9,10 +9,10 @@
     <xacro:property name="wheel_thickness" value="0.028"/>
     <xacro:property name="wheel_mass" value="0.05"/>
-    <xacro:property name="wheel_offset_x" value="0.145"/>
+    <xacro:property name="wheel_offset_x" value="0.0238"/>
     <xacro:property name="wheel_offset_y" value="0.0675"/>
     <xacro:property name="wheel_offset_z" value="0.035"/>
     <xacro:property name="caster_wheel_radius" value="0.033"/>
     <xacro:property name="caster_wheel_mass" value="0.01"/>
-    <xacro:property name="caster_wheel_offset_x" value="0.025"/>
+    <xacro:property name="caster_wheel_offset_x" value="0.1438"/>
     <!-- <xacro:property name="caster_wheel_offset_z" value="${wheel_offset_z - wheel_radius + caster_wheel_radius}"/> -->
     <xacro:property name="caster_wheel_offset_z" value="${-caster_wheel_radius}"/>

Commit message: change the color wheel and chassis in gazebo

File: description/robot_core.xacro (robot description, xacro)
@@ -74,5 +74,5 @@
     </link>
     <gazebo reference="chassis">
-        <material>Gazebo/Orange</material>
+        <material>Gazebo/Green</material>
     </gazebo>
     <!-- LEFT WHEEL LINK -->
@@ -100,5 +100,5 @@
     </link>
     <gazebo reference="left_wheel">
-        <material>Gazebo/Blue</material>
+        <material>Gazebo/Yellow</material>
     </gazebo>
     <!-- RIGHT WHEEL LINK -->
@@ -126,5 +126,5 @@
     </link>
     <gazebo reference="right_wheel">
-        <material>Gazebo/Blue</material>
+        <material>Gazebo/Yellow</material>
     </gazebo>
     <!-- CASTER WHEEL LINK -->
