Commit message: try to implement a slam with slam_toolbox

File: description/lidar.xacro (robot description, xacro)
@@ -45,5 +45,5 @@
                 <range>
                     <min>0.3</min>
-                    <max>12</max>
+                    <max>2.0</max>
                 </range>
             </ray>

File: description/robot.urdf.xacro (robot description, xacro)
@@ -4,6 +4,18 @@
     <xacro:include filename="robot_core.xacro" />
     <xacro:include filename="gazebo_control.xacro" />
-    <!-- <xacro:include filename="lidar.xacro" /> -->
-    <xacro:include filename="sonar.xacro" />
+    <!-- <xacro:include filename="sonar.xacro" /> -->
+     <!-- <xacro:if value="$(arg use_ros2_control)">
+        <xacro:include filename="ros2_control.xacro" />
+    </xacro:if>
+    <xacro:unless value="$(arg use_ros2_control)">
+        <xacro:include filename="gazebo_control.xacro" />
+    </xacro:unless> -->
+    <xacro:include filename="lidar.xacro" />
+    <!-- <xacro:if value="$(arg robot_simulation)">
+        <xacro:include filename="lidar.xacro" />
+    </xacro:if>
+    <xacro:unless value="$(arg robot_simulation)">
+        <xacro:include filename="sonar.xacro" />
+    </xacro:unless> -->
     <!-- <link name="base_link"></link> -->
 </robot>

File: description/sonar.xacro (robot description, xacro)
@@ -25,3 +25,28 @@
       </collision>
     </link>
+    <gazebo reference="sonar_link">
+        <material>Gazebo/Blue</material>
+        <sensor name="laser" type="ray">
+            <pose> 0 0 0 0 0 0 </pose>
+            <visualize>false</visualize>
+            <update_rate>10</update_rate>
+            <ray>
+                <scan>
+                    <horizontal>
+                        <samples>6</samples>
+                        <min_angle>-1.0</min_angle>
+                        <max_angle>1.0</max_angle>
+                    </horizontal>
+                </scan>
+                <range>
+                    <min>0.3</min>
+                    <max>2.0</max>
+                </range>
+            </ray>
+            <plugin name="laser_controller" filename="libgazebo_ros_ray_sensor.so">
+                <output_type>sensor_msgs/LaserScan</output_type>
+                <frame_name>sonar_link</frame_name>
+            </plugin>
+        </sensor>
+    </gazebo>
 </robot>
