Commit message: add lidar.xacro file sonar.xacro file for LaserScan message

File: description/robot.urdf.xacro (robot description, xacro)
@@ -4,4 +4,6 @@
     <xacro:include filename="robot_core.xacro" />
     <xacro:include filename="gazebo_control.xacro" />
+    <!-- <xacro:include filename="lidar.xacro" /> -->
+    <xacro:include filename="sonar.xacro" />
     <!-- <link name="base_link"></link> -->
 </robot>

File: description/robot_core.xacro (robot description, xacro)
@@ -8,10 +8,10 @@
     <xacro:property name="wheel_radius" value="0.033"/>
     <xacro:property name="wheel_thickness" value="0.028"/>
-    <xacro:property name="wheel_mass" value="0.05"/>
+    <xacro:property name="wheel_mass" value="0.3"/>
     <xacro:property name="wheel_offset_x" value="0.0238"/>
     <xacro:property name="wheel_offset_y" value="0.0675"/>
     <xacro:property name="wheel_offset_z" value="0.035"/>
     <xacro:property name="caster_wheel_radius" value="0.033"/>
-    <xacro:property name="caster_wheel_mass" value="0.01"/>
+    <xacro:property name="caster_wheel_mass" value="5"/>
     <xacro:property name="caster_wheel_offset_x" value="0.1438"/>
     <!-- <xacro:property name="caster_wheel_offset_z" value="${wheel_offset_z - wheel_radius + caster_wheel_radius}"/> -->

Commit message: add a sonar sensor to the rviz and add sonar nodes to launch files

File: description/robot.urdf.xacro (robot description, xacro)
@@ -3,6 +3,6 @@
     <!-- Example link -->
     <xacro:include filename="robot_core.xacro" />
-    <xacro:include filename="gazebo_control.xacro" />
-    <!-- <xacro:include filename="sonar.xacro" /> -->
+    <!-- <xacro:include filename="gazebo_control.xacro" /> -->
+    <xacro:include filename="sonar.xacro" />
      <!-- <xacro:if value="$(arg use_ros2_control)">
         <xacro:include filename="ros2_control.xacro" />
@@ -11,5 +11,5 @@
         <xacro:include filename="gazebo_control.xacro" />
     </xacro:unless> -->
-    <xacro:include filename="lidar.xacro" />
+    <!-- <xacro:include filename="lidar.xacro" /> -->
     <!-- <xacro:if value="$(arg robot_simulation)">
         <xacro:include filename="lidar.xacro" />

File: description/sonar.xacro (robot description, xacro)
@@ -25,28 +25,3 @@
       </collision>
     </link>
-    <gazebo reference="sonar_link">
-        <material>Gazebo/Blue</material>
-        <sensor name="laser" type="ray">
-            <pose> 0 0 0 0 0 0 </pose>
-            <visualize>false</visualize>
-            <update_rate>10</update_rate>
-            <ray>
-                <scan>
-                    <horizontal>
-                        <samples>6</samples>
-                        <min_angle>-1.0</min_angle>
-                        <max_angle>1.0</max_angle>
-                    </horizontal>
-                </scan>
-                <range>
-                    <min>0.3</min>
-                    <max>2.0</max>
-                </range>
-            </ray>
-            <plugin name="laser_controller" filename="libgazebo_ros_ray_sensor.so">
-                <output_type>sensor_msgs/LaserScan</output_type>
-                <frame_name>sonar_link</frame_name>
-            </plugin>
-        </sensor>
-    </gazebo>
 </robot>
